Commit message: Rename indy7

File: example/indy7/indy7/indy7.urdf (robot description, URDF)
Before this commit: robot indy7, 9 links, 8 joints
Links:
- link base_link: geometry collision cylinder length=0.075 radius=0.102; visual mesh filename=visual/Indy7_0.stl
- link forearm_link: geometry collision cylinder length=0.075 radius=0.045; collision cylinder length=0.267 radius=0.045
- link shoulder_link: geometry collision cylinder length=0.109 radius=0.075; collision cylinder length=0.222 radius=0.075
- link upper_arm_link: geometry collision cylinder length=0.09 radius=0.075; collision cylinder length=0.1205 radius=0.045
- link wrist_1_link: geometry collision cylinder length=0.083 radius=0.045; collision cylinder length=0.114 radius=0.045
- link wrist_2_link: geometry collision cylinder length=0.069 radius=0.045; collision cylinder length=0.168 radius=0.045
- link wrist_3_link: geometry collision cylinder length=0.06 radius=0.045; visual mesh filename=visual/Indy7_6.stl
