Commit message: Add franka vis

File: example/franka/panda_arm.urdf (robot description, URDF)
Before this commit: robot panda_arm, 9 links, 8 joints
Links:
- link panda_link0: geometry collision mesh filename=package://meshes/collision/link0.obj; visual mesh filename=package://meshes/collision/link0.obj
- link panda_link1: geometry collision mesh filename=package://meshes/collision/link1.obj; visual mesh filename=package://meshes/visual/link1.obj
- link panda_link2: geometry collision mesh filename=package://meshes/collision/link2.obj; visual mesh filename=package://meshes/visual/link2.obj
- link panda_link3: geometry collision mesh filename=package://meshes/collision/link3.obj; visual mesh filename=package://meshes/visual/link3.obj
- link panda_link4: geometry collision mesh filename=package://meshes/collision/link4.obj; visual mesh filename=package://meshes/visual/link4.obj
- link panda_link5: geometry collision mesh filename=package://meshes/collision/link5.obj; visual mesh filename=package://meshes/visual/link5.obj
- link panda_link6: geometry collision mesh filename=package://meshes/collision/link6.obj; visual mesh filename=package://meshes/visual/link6.obj
- link panda_link7: geometry collision mesh filename=package://meshes/collision/link7.obj; visual mesh filename=package://meshes/collision/link7.obj
